File: 6 Meter Tranciever Kicad/RF Pre Amp/RF Pre Amp.sch (KiCad schematic (older format))
At the start: 52 parts, among them J1 RF In, J2 RF Out, J3 Conn_01x03_Male, J4 Conn_01x03_Male, Q1 BFR106, Q10 BFR106, Q2 BFR106, Q3 AO3400A, Q4 AO3401A, Q5 BFR106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

Commit message: Board tweaks
Board tweaks and remove bak files
Parts:
- removed C12: 33n, WC8C:SMD_Combo_1206_0805, symbol Device:C_Small
Changed lines of the file:
@@
 	0    1    -1   0
 $EndComp
-$Comp
-L Device:C_Small C12
-U 1 1 622AA91A
-P 1150 3700
-F 0 "C12" H 900 3750 50  0000 L CNN
-F 1 "33n" H 900 3650 50  0000 L CNN
-F 2 "WC8C:SMD_Combo_1206_0805" H 1150 3700 50  0001 C CNN
-F 3 "~" H 1150 3700 50  0001 C CNN
-	1    1150 3700
-	1    0    0    -1
-$EndComp
-Wire Wire Line
-	1600 3400 1150 3400
-Wire Wire Line
-	1150 3400 1150 3600
-Wire Wire Line
-	1600 3950 1150 3950
-Wire Wire Line
-	1150 3950 1150 3800
-Connection ~ 1600 3950
 $EndSCHEMATC
