File: 6 Meter Tranciever Kicad/TermionationInsensitiveAmplifier/TerminationInsensitiveAmplifier.kicad_pcb (KiCad board)
At the start: 2 copper layers, 66.2 x 61.3 mm, 97 parts, among them J1 Power & RX/TX, J2 PWR, J3 TX In / RX Out, J4 RX IN / TX Out, J5 Jumper, J6 Jumper, J7 Power & RX/TX, J8 GND TP, J80 Audio, J81 Audio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

Commit message: Board tweaks
Board tweaks and remove bak files
Parts:
- removed C16: 33n, WC8C:SMD_Combo_1206_0805
- moved R87 20.7 mm to (167.0, 85.0)
- moved R88 12.8 mm to (175.1, 94.8)
- moved R80 3.34 mm to (129.6, 80.7), turned to 0 degrees
- moved R28 1.49 mm to (134.6, 80.7)
- moved C10 1.40 mm to (168.9, 79.5)
- moved C1 0.97 mm to (166.8, 71.2)
- moved R5 0.36 mm to (156.4, 82.1)
- moved R4 0.21 mm to (161.3, 79.6)
Routing:
- net GNDREF: track 259.2 -> 229.5 mm
- net Net-(C85-Pad1): track 66.5 -> 70.0 mm
- net Net-(C6-Pad2): track 11.7 -> 15.0 mm
- net /RX_Low_TX_High: track 28.3 -> 25.7 mm
- net Net-(C5-Pad1): track 30.6 -> 32.9 mm
- net Net-(C10-Pad1): track 4.19 -> 5.65 mm
- net Net-(C10-Pad2): track 22.8 -> 24.0 mm
- net Net-(C11-Pad1): track 47.1 -> 48.1 mm
- net Net-(Q10-Pad1): track 10.5 -> 11.3 mm
- net Net-(C1-Pad2): track 14.8 -> 15.4 mm
