File: 6 Meter Tranciever Kicad/TermionationInsensitiveAmplifier/TerminationInsensitiveAmplifier.sch (KiCad schematic (older format))
At the start: 89 parts, among them J1 Power & RX/TX, J2 PWR, J3 TX In / RX Out, J4 RX IN / TX Out, J5 Jumper, J6 Jumper, J7 Power & RX/TX, J8 GND TP, J80 Audio, J81 Audio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

Commit message: Board tweaks
Board tweaks and remove bak files
Parts:
- removed C16: 33n, WC8C:SMD_Combo_1206_0805, symbol Device:C
Changed lines of the file:
@@
 	1    0    0    -1
 $EndComp
-Wire Wire Line
-	1750 4500 2150 4500
 $Comp
 L power:GNDREF #PWR0108
@@
 Wire Wire Line
 	7200 2300 7400 2300
-$Comp
-L Device:C C16
-U 1 1 622E15DD
-P 2150 4700
-F 0 "C16" H 2265 4746 50  0000 L CNN
-F 1 "33n" H 2265 4655 50  0000 L CNN
-F 2 "WC8C:SMD_Combo_1206_0805" H 2188 4550 50  0001 C CNN
-F 3 "~" H 2150 4700 50  0001 C CNN
-	1    2150 4700
-	1    0    0    -1
-$EndComp
-Connection ~ 2150 4500
-Wire Wire Line
-	2550 4900 2150 4900
-Wire Wire Line
-	2150 4500 2550 4500
-Connection ~ 2550 4900
-Wire Wire Line
-	2150 4550 2150 4500
-Wire Wire Line
-	2150 4900 2150 4850
+Wire Wire Line
+	1750 4500 2550 4500
 $EndSCHEMATC
